Commit message: first commit

File: catvehicle_basics/catvehicle/urdf/catvehicle_mod.xacro (robot description, xacro)
@@ -1,3 +1,3 @@
-<?xml version="1.0" ?>
+<?xml version="1.0" encoding="UTF-8"?>
 <!--
 Author: Jonathan Sprinkle, Sam Taylor, Alex Warren
@@ -26,642 +26,546 @@
 roslaunch catvehicle catvehicle_skidpan.launch
 -->
+<!--
+Modified by : Amirmohammad Zarif
+Copyright (c) 2021
+-->
 <!-- Inertial parameters selected with the help of
 http://www.car-engineer.com/vehicle-inertia-calculation-tool/
 -->
-<robot name="$(arg roboname)" xmlns:xacro="http://www.ros.org/wiki/xacro">
-  <xacro:arg name="camera_left" default="false"/>
-  <xacro:arg name="camera_right" default="false"/>
-  <xacro:arg name="camera_front" default="true"/>
-  <xacro:arg name="camera_back" default="false"/>
-  <xacro:arg name="velodyne_points" default="true"/>
-  <xacro:arg name="front_laser_points" default="true"/>
-  <xacro:property name="PI" value="3.1415926835897931"/>
-  <xacro:property name="base_height" value="1.0639"/>
-  <xacro:property name="base_collision_height" value="1.3639"/>
-  <xacro:property name="base_mass" value="2050"/>
-  <xacro:property name="base_mass_ixx" value="647"/>
-  <xacro:property name="base_mass_iyy" value="3291"/>
-  <xacro:property name="base_mass_izz" value="3360"/>
-  <xacro:property name="base_mass_ixz" value="-31"/>
-  <xacro:property name="tyre_x" value="1.41"/>
-  <xacro:property name="tyre_y" value="0.765"/>
-  <xacro:property name="tyre_length" value="0.229"/>
-  <xacro:property name="tyre_r" value="0.66"/>
-  <xacro:property name="tyre_radius" value="0.356"/>
-  <xacro:property name="tyre_mass" value="40"/>
- <xacro:property name="tyre_mass_ixx" value="2.0"/>
-  <xacro:property name="tyre_mass_iyy" value="2.0"/>
-  <xacro:property name="tyre_mass_izz" value="2.0"/>
-  <xacro:property name="car_height" value="1.4478"/>
-  <xacro:property name="car_to_bumper" value="2.4"/>
-  <xacro:property name="front_bumper_height" value="${car_height/2}"/>
-  <xacro:property name="sensor_box" value="0.25"/>
-  <xacro:property name="sensor_box2" value="0.01"/>
-  <xacro:property name="camera_box" value="0.1"/>
-  <xacro:property name="tyre_height" value="-0.696"/>
-  <xacro:property name="str_length" value="0.01"/>
-  <xacro:property name="str_radius" value="0.1"/>
-  <xacro:property name="str_angle" value="0.6"/>
-  <xacro:property name="car_width" value="1.301"/>
-  <xacro:property name="front_laser_points" value="$(arg front_laser_points)"/>
-  <xacro:property name="velodyne_points" value="$(arg velodyne_points)"/>
-  <xacro:property name="camera_right" value="$(arg camera_right)"/>
-  <xacro:property name="camera_left" value="$(arg camera_left)"/>
-  <xacro:property name="camera_front" value="$(arg camera_front)"/>
-  <xacro:property name="camera_back" value="$(arg camera_back)"/>
-  <xacro:property name="tyre_origin">
-	<origin xyz="0 0 0" rpy="${PI/2} 0 0"/>
-  </xacro:property>
-  <xacro:property name="tyre_origin_2">
-        <origin xyz="0 0 0" rpy="0 0 ${PI/2}"/>
-  </xacro:property>
-  <xacro:property name="tyre_origin_3">
-        <origin xyz="0 0 0" rpy="0 0 ${-PI/2}"/>
-  </xacro:property>
-	<!--<xacro:include filename="$(find catvehicle)/urdf/catvehicle.gazebo"/>-->
+<robot xmlns:xacro="http://www.ros.org/wiki/xacro" name="$(arg roboname)">
+    <xacro:arg name="camera_left" default="false" />
+    <xacro:arg name="camera_right" default="false" />
+    <xacro:arg name="camera_front" default="true" />
+    <xacro:arg name="camera_back" default="false" />
+    <xacro:arg name="velodyne_points" default="true" />
+    <xacro:arg name="front_laser_points" default="true" />
+    <xacro:property name="PI" value="3.1415926835897931" />
+    <xacro:property name="base_height" value="1.0639" />
+    <xacro:property name="base_collision_height" value="1.3639" />
+    <xacro:property name="base_mass" value="2050" />
+    <xacro:property name="base_mass_ixx" value="647" />
+    <xacro:property name="base_mass_iyy" value="3291" />
+    <xacro:property name="base_mass_izz" value="3360" />
+    <xacro:property name="base_mass_ixz" value="-31" />
+    <xacro:property name="tyre_x" value="1.41" />
+    <xacro:property name="tyre_y" value="0.765" />
+    <xacro:property name="tyre_length" value="0.229" />
+    <xacro:property name="tyre_r" value="0.66" />
+    <xacro:property name="tyre_radius" value="0.356" />
+    <xacro:property name="tyre_mass" value="40" />
+    <xacro:property name="tyre_mass_ixx" value="2.0" />
+    <xacro:property name="tyre_mass_iyy" value="2.0" />
+    <xacro:property name="tyre_mass_izz" value="2.0" />
+    <xacro:property name="car_height" value="1.4478" />
+    <xacro:property name="car_to_bumper" value="2.4" />
+    <xacro:property name="front_bumper_height" value="${car_height/2}" />
+    <xacro:property name="sensor_box" value="0.25" />
+    <xacro:property name="sensor_box2" value="0.01" />
+    <xacro:property name="camera_box" value="0.1" />
+    <xacro:property name="tyre_height" value="-0.696" />
+    <xacro:property name="str_length" value="0.01" />
+    <xacro:property name="str_radius" value="0.1" />
+    <xacro:property name="str_angle" value="0.6" />
+    <xacro:property name="car_width" value="1.301" />
+    <xacro:property name="front_laser_points" value="$(arg front_laser_points)" />
+    <xacro:property name="velodyne_points" value="$(arg velodyne_points)" />
+    <xacro:property name="camera_right" value="$(arg camera_right)" />
+    <xacro:property name="camera_left" value="$(arg camera_left)" />
+    <xacro:property name="camera_front" value="$(arg camera_front)" />
+    <xacro:property name="camera_back" value="$(arg camera_back)" />
+    <xacro:property name="tyre_origin">
+        <origin xyz="0 0 0" rpy="${PI/2} 0 0" />
+    </xacro:property>
+    <xacro:property name="tyre_origin_2">
+        <origin xyz="0 0 0" rpy="0 0 ${PI/2}" />
+    </xacro:property>
+    <xacro:property name="tyre_origin_3">
+        <origin xyz="0 0 0" rpy="0 0 ${-PI/2}" />
+    </xacro:property>
+    <!--<xacro:include filename="$(find catvehicle)/urdf/catvehicle.gazebo"/>-->
     <xacro:if value="${front_laser_points}">
-    	<xacro:include filename="$(find catvehicle)/urdf/catvehicle_front_laser_points.gazebo"/>
+        <xacro:include filename="$(find catvehicle)/urdf/catvehicle_front_laser_points.gazebo" />
     </xacro:if>
     <xacro:if value="${velodyne_points}">
-      <!-- You can pass parameters in order to change the max/min
+        <!-- You can pass parameters in order to change the max/min
            horizontal angles of the velodyne sensors. These are interpreted
            in the velodyne_points gazebo file -->
-      <xacro:arg name="velodyne_min_angle" default="-0.4"/>
-      <xacro:arg name="velodyne_max_angle" default="0.4"/>
-      <xacro:property name="velodyne_min_angle" value="$(arg velodyne_min_angle)"/>
-      <xacro:property name="velodyne_max_angle" value="$(arg velodyne_max_angle)"/>
-    	<xacro:include filename="$(find catvehicle)/urdf/catvehicle_velodyne_points.gazebo"/>
+        <xacro:arg name="velodyne_min_angle" default="-0.4" />
+        <xacro:arg name="velodyne_max_angle" default="0.4" />
+        <xacro:property name="velodyne_min_angle" value="$(arg velodyne_min_angle)" />
+        <xacro:property name="velodyne_max_angle" value="$(arg velodyne_max_angle)" />
+        <xacro:include filename="$(find catvehicle)/urdf/catvehicle_velodyne_points.gazebo" />
     </xacro:if>
     <xacro:if value="${camera_right}">
-    	<xacro:include filename="$(find catvehicle)/urdf/catvehicle_right_camera.gazebo"/>
+        <xacro:include filename="$(find catvehicle)/urdf/catvehicle_right_camera.gazebo" />
     </xacro:if>
     <xacro:if value="${camera_left}">
-    	<xacro:include filename="$(find catvehicle)/urdf/catvehicle_left_camera.gazebo"/>
+        <xacro:include filename="$(find catvehicle)/urdf/catvehicle_left_camera.gazebo" />
     </xacro:if>
     <xacro:if value="${camera_front}">
-    	<xacro:include filename="$(find catvehicle)/urdf/catvehicle_front_camera.gazebo"/>
+        <xacro:include filename="$(find catvehicle)/urdf/catvehicle_front_camera.gazebo" />
     </xacro:if>
     <xacro:if value="${camera_back}">
-    	<xacro:include filename="$(find catvehicle)/urdf/catvehicle_back_camera.gazebo"/>
+        <xacro:include filename="$(find catvehicle)/urdf/catvehicle_back_camera.gazebo" />
     </xacro:if>
-<!--Car Body-->
-<link name="base_link">
-    <collision>
-         <origin xyz="0 0 ${base_collision_height}" rpy="0 0 0"/>
-           <geometry>
-            <box size="4.192 ${car_width} ${car_height}"/>
-        </geometry>
-      </collision>
-     <visual>
-        <origin xyz="-0.25 0 ${base_height + 0.05}" rpy="0 0 0"/>
-        <geometry>
-          <!--<mesh filename="package://catvehicle/meshes/ford_escape_no_wheels_2.dae"/>-->
-          <mesh filename="package://catvehicle/meshes/udemy_car_simplified_v2.dae"/>
-          <!--<box size="4.192 ${car_width} ${car_height}"/>-->
-        </geometry>
-     </visual>
-</link>
-<joint name="inertial_joint" type="fixed">
-      <parent link="base_link"/>
-      <child link="main_mass"/>
-      <origin xyz="0 0 0" rpy="0 0 0"/>
-</joint>
-<link name="main_mass" type="fixed">
-     <parent link="inertial_joint"/>
-     <inertial>
-        <origin xyz="0 0 ${base_height}" rpy="0 0 0"/>
-        <mass value="${base_mass}"/>
-        <inertia
-          ixx="${base_mass_ixx}"  ixy="0.000000" ixz="${base_mass_ixz}"
-          iyy="${base_mass_iyy}" iyz="0.000000"
-          izz="${base_mass_izz}"/>
-      </inertial>
-</link>
-<!--Back Right Wheel-->
-<joint name="back_right_wheel_joint" type="continuous">
-      <parent link="base_link"/>
-      <child link="back_right_wheel_link"/>
-      <origin xyz="${-tyre_x} ${-tyre_y} ${tyre_r}" rpy="0 0 0"/>
-      <axis xyz="0 1 0"/>
-      <dynamics damping="0.1"/>
-     <!--<limit effort="10000" velocity="100" />-->
-     <limit effort="100000" velocity="10000" />
-      <joint_properties damping="0.0" friction="0.0" />
-</joint>
-<link name="back_right_wheel_link">
-     <collision>
-      <xacro:insert_block name="tyre_origin"/>
-        <geometry>
-         <cylinder length="${tyre_length}" radius="${tyre_radius}"/>
-        </geometry>
-     </collision>
-     <visual>
-      <xacro:insert_block name="tyre_origin_3"/>
-        <geometry>
-          <!--<mesh filename="package://catvehicle/meshes/ford_escape_wheel.dae"/>-->
-          <mesh filename="package://catvehicle/meshes/wheel_simplified_v3.dae"/>
-          <!--<cylinder length="${tyre_length}" radius="${tyre_radius}"/>-->
-          <!--<box size="${tyre_r} ${tyre_r} ${tyre_length}"/>-->
-      <scale xyz="1.2 1 1"/>
-        </geometry>
-      </visual>
-      <inertial>
-        <origin xyz="0 0 0" rpy="0 0 0"/>
-        <mass value="${tyre_mass}"/>
-        <inertia
-          ixx="${tyre_mass_ixx}"  ixy="0.000000"  ixz="0.000000"
-          iyy="${tyre_mass_iyy}"  iyz="0.000000"
-          izz="${tyre_mass_izz}"/>
-      </inertial>
-</link>
-<!--Back Left Wheel-->
-<joint name="back_left_wheel_joint" type="continuous">
-      <parent link="base_link"/>
-      <child link="back_left_wheel_link"/>
-      <origin xyz="${-tyre_x} ${tyre_y} ${tyre_r}" rpy="0 0 0"/>
-      <axis xyz="0 1 0"/>
-      <dynamics damping="0.1"/>
-      <!--<limit effort="10000" velocity="100" />-->
-      <limit effort="100000" velocity="10000" />
-      <joint_properties damping="0.0" friction="0.0" />
-</joint>
-<link name="back_left_wheel_link">
-     <collision>
-      <xacro:insert_block name="tyre_origin"/>
-        <geometry>
-         <cylinder length="0.229" radius="${tyre_radius}"/>
-        </geometry>
-     </collision>
-     <visual>
-      <xacro:insert_block name="tyre_origin_2"/>
-        <geometry>
-          <!--<mesh filename="package://catvehicle/meshes/ford_escape_wheel.dae"/>-->
-          <mesh filename="package://catvehicle/meshes/wheel_simplified_v3.dae"/>
-          <!--<cylinder length="${tyre_length}" radius="${tyre_radius}"/>-->
-          <!--<box size="${tyre_r} ${tyre_r} ${tyre_length}"/>-->
-          <scale xyz="1.2 1 1"/>
-        </geometry>
-      </visual>
-      <inertial>
-        <origin xyz="0 0 0" rpy="0 0 0"/>
-        <mass value="${tyre_mass}"/>
-        <inertia
-          ixx="${tyre_mass_ixx}"  ixy="0.000000"  ixz="0.000000"
-          iyy="${tyre_mass_iyy}"  iyz="0.000000"
-          izz="${tyre_mass_izz}"/>
-      </inertial>
-</link>
-<!--Right Steering-->
-<joint name="front_right_steering_joint" type="revolute">
-	<parent link="base_link"/>
-	<child link="front_right_steering_link"/>
-	<origin xyz="${tyre_x} ${-car_width/2 - str_length/2} ${tyre_r}" rpy="0 0 0"/>
-    <axis xyz="0 0 1"/>
-	<limit lower="${-str_angle}" upper="${str_angle}" effort="1000000.0" velocity="10000.0"/>
-	<dynamics damping="100"/>
-</joint>
-<link name="front_right_steering_link">
-	<collision>
-	      <xacro:insert_block name="tyre_origin"/>
-	        <geometry>
-        	 <cylinder length="${str_length}" radius="${str_radius}"/>
-       		</geometry>
-	</collision>
-	<visual>
-              <xacro:insert_block name="tyre_origin"/>
-                <geometry>
-                 <cylinder length="${str_length}" radius="${str_radius}"/>
-                </geometry>
-	</visual>
-      <inertial>
-        <origin xyz="0 0 0" rpy="0 0 0"/>
-        <mass value="10.00"/>
-        <inertia
-          ixx="0.4"  ixy="0.000000"  ixz="0.000000"
-          iyy="0.6"  iyz="0.000000"
-          izz="0.4"/>
-      </inertial>
-</link>
-<!--Right Front Wheel-->
-<joint name="front_right_wheel_joint" type="continuous">
-      <parent link="front_right_steering_link"/>
-      <child link="front_right_wheel_link"/>
-      <origin xyz="0 ${-str_length/2 - tyre_length/2} 0" rpy="0 0 0"/>
-      <axis xyz="0 1 0"/>
-      <dynamics damping="0.1"/>
-     <!--<limit effort="10000" velocity="100" />-->
-     <limit effort="1000000" velocity="10000" />
-      <joint_properties damping="0.0" friction="0.0" />
-</joint>
-<link name="front_right_wheel_link">
-     <collision>
-      <xacro:insert_block name="tyre_origin"/>
-        <geometry>
-         <cylinder length="${tyre_length}" radius="${tyre_radius}"/>
-	</geometry>
-     </collision>
-     <visual>
-      <xacro:insert_block name="tyre_origin_3"/>
-        <geometry>
-          <!--<mesh filename="package://catvehicle/meshes/ford_escape_wheel.dae"/>-->
-          <mesh filename="package://catvehicle/meshes/wheel_simplified_v3.dae"/>
-          <!--<cylinder length="${tyre_length}" radius="${tyre_radius}"/>-->
-          <!--<box size="${tyre_r} ${tyre_r} ${tyre_length}"/>-->
-        <scale xyz="1.2 1 1"/>
-       </geometry>
-      </visual>
-      <inertial>
-        <origin xyz="0 0 0" rpy="0 0 0"/>
-        <mass value="${tyre_mass}"/>
-        <inertia
-          ixx="${tyre_mass_ixx}"  ixy="0.000000"  ixz="0.000000"
-          iyy="${tyre_mass_iyy}"  iyz="0.000000"
-          izz="${tyre_mass_izz}"/>
-      </inertial>
-</link>
-<!--Left Steering-->
-<joint name="front_left_steering_joint" type="revolute">
-        <parent link="base_link"/>
-        <child link="front_left_steering_link"/>
-        <origin xyz="${tyre_x} ${car_width/2 + str_length/2} ${tyre_r}" rpy="0 0 0"/>
-        <axis xyz="0 0 1"/>
-        <limit lower="${-str_angle}" upper="${str_angle}" effort="1000000.0" velocity="10000.0"/>
+    <!--Car Body-->
+    <link name="base_link">
+        <collision>
+            <origin xyz="0 0 ${base_collision_height}" rpy="0 0 0" />
+            <geometry>
+                <box size="4.192 ${car_width} ${car_height}" />
+            </geometry>
+        </collision>
+        <visual>
+            <origin xyz="-0.25 0 ${base_height + 0.05}" rpy="0 0 0" />
+            <geometry>
+                <!--<mesh filename="package://catvehicle/meshes/ford_escape_no_wheels_2.dae"/>-->
+                <!-- <mesh filename="package://catvehicle/meshes/udemy_car_simplified_v2.dae"/> -->
+                <mesh filename="package://catvehicle/meshes/mesh_avis_audi_car_simplified.dae" />
+                <!--<box size="4.192 ${car_width} ${car_height}"/>-->
+            </geometry>
+        </visual>
+    </link>
+    <joint name="inertial_joint" type="fixed">
+        <parent link="base_link" />
+        <child link="main_mass" />
+        <origin xyz="0 0 0" rpy="0 0 0" />
+    </joint>
+    <link name="main_mass" type="fixed">
+        <parent link="inertial_joint" />
+        <inertial>
+            <origin xyz="0 0 ${base_height}" rpy="0 0 0" />
+            <mass value="${base_mass}" />
+            <inertia ixx="${base_mass_ixx}" ixy="0.000000" ixz="${base_mass_ixz}" iyy="${base_mass_iyy}" iyz="0.000000" izz="${base_mass_izz}" />
+        </inertial>
+    </link>
+    <!--Back Right Wheel-->
+    <joint name="back_right_wheel_joint" type="continuous">
+        <parent link="base_link" />
+        <child link="back_right_wheel_link" />
+        <origin xyz="${-tyre_x} ${-tyre_y} ${tyre_r}" rpy="0 0 0" />
+        <axis xyz="0 1 0" />
+        <dynamics damping="0.1" />
+        <!--<limit effort="10000" velocity="100" />-->
+        <limit effort="100000" velocity="10000" />
+        <joint_properties damping="0.0" friction="0.0" />
+    </joint>
+    <link name="back_right_wheel_link">
+        <collision>
+            <xacro:insert_block name="tyre_origin" />
+            <geometry>
+                <cylinder length="${tyre_length}" radius="${tyre_radius}" />
+            </geometry>
+        </collision>
+        <visual>
+            <xacro:insert_block name="tyre_origin_3" />
+            <geometry>
+                <!--<mesh filename="package://catvehicle/meshes/ford_escape_wheel.dae"/>-->
+                <!-- <mesh filename="package://catvehicle/meshes/wheel_simplified_v3.dae"/> -->
+                <mesh filename="package://catvehicle/meshes/mesh_avis_small_wheel_simplified.dae" />
+                <!--<cylinder length="${tyre_length}" radius="${tyre_radius}"/>-->
+                <!--<box size="${tyre_r} ${tyre_r} ${tyre_length}"/>-->
+                <scale xyz="1.2 1 1" />
+            </geometry>
+        </visual>
+        <inertial>
+            <origin xyz="0 0 0" rpy="0 0 0" />
+            <mass value="${tyre_mass}" />
+            <inertia ixx="${tyre_mass_ixx}" ixy="0.000000" ixz="0.000000" iyy="${tyre_mass_iyy}" iyz="0.000000" izz="${tyre_mass_izz}" />
+        </inertial>
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